File: Gitclock/Gitclock.kicad_sch (KiCad schematic)
At the start: 41 parts, among them J1 PJ-102AH, J2 Conn_01x06, J3 Conn_01x05, SW1 Omron_B3F_SPST, SW2 Omron_B3F_SPST, SW3 Omron_B3F_SPST, SW4 Omron_B3F_SPST, SW5 RotaryEncoder_Switch, U1 ATmega328-PU, U2 L7805, U3 MAX7219, U4 DS1307_DIP-8, U5 ULN2003A, Y1 Crystal_16MHz, Y2 Crystal_32768Hz

Commit message: Updatedclock
20220705
6:27PM
Parts:
- added RV2: R_POT_10K, footprints:Potentiometer_Bourns_3386P_Vertical, symbol HPS:R_POT_10K
Connections:
- net BUZZER: now also BZ1.2 (+)
- net FAN: no longer BZ1.2 (+)
- net SCL: no longer SW5.A
- net MENU OUTPUT2: now reaches U1.23 (PC0)
- net MENU OUTPUT2: now also SW5.A
- net at DS2.3 (VO): now also RV2.1
- no-connect marks 25 -> 37
Changed lines of the file:
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@@
   (no_connect (at 38.1 118.11))
   (no_connect (at 50.8 231.14))
+  (no_connect (at 115.57 58.42))
+  (no_connect (at 115.57 60.96))
+  (no_connect (at 45.72 220.98))
+  (no_connect (at 35.56 220.98))
+  (no_connect (at 52.07 50.8))
+  (no_connect (at -44.45 233.68))
+  (no_connect (at 378.46 59.69))
+  (no_connect (at 388.62 59.69))
+  (no_connect (at 377.19 27.94))
+  (no_connect (at 387.35 27.94))
+  (no_connect (at 198.12 149.86))
+  (no_connect (at 198.12 152.4))
   (no_connect (at 213.36 60.96))
   (wire (pts (xy 67.31 48.26) (xy 67.31 20.32))
@@
     (stroke (width 0) (type default) (color 0 0 0 0))
   )
-  (polyline (pts (xy 389.89 137.16) (xy 367.03 137.16))
+  (polyline (pts (xy 393.7 137.16) (xy 367.03 137.16))
     (stroke (width 0) (type default) (color 0 0 0 0))
   )
@@
     (stroke (width 0) (type default) (color 0 0 0 0))
   )
-  (polyline (pts (xy 367.03 111.76) (xy 389.89 111.76))
+  (polyline (pts (xy 367.03 111.76) (xy 393.7 111.76))
     (stroke (width 0) (type default) (color 0 0 0 0))
   )
@@
     (stroke (width 0) (type default) (color 0 0 0 0))
   )
-  (polyline (pts (xy 389.89 111.76) (xy 389.89 137.16))
+  (polyline (pts (xy 393.7 111.76) (xy 393.7 137.16))
     (stroke (width 0) (type default) (color 0 0 0 0))
   )
@@
     )
   )
+  (global_label "MENU OUTPUT2" (shape output) (at 198.12 144.78 0) (fields_autoplaced)
+    (effects (font (size 1.27 1.27)) (justify left))
+    (property "Intersheet References" "${INTERSHEET_REFS}" (id 0) (at 215.1683 144.7006 0)
+      (effects (font (size 1.27 1.27)) (justify left) hide)
+    )
+  )
   (global_label "SDA" (shape output) (at 203.2 154.94 0) (fields_autoplaced)
     (effects (font (size 1.27 1.27)) (justify left))
@@
     )
   )
+  (global_label "MENU OUTPUT2" (shape input) (at 370.84 97.79 180) (fields_autoplaced)
+    (effects (font (size 1.27 1.27)) (justify right))
+    (property "Intersheet References" "${INTERSHEET_REFS}" (id 0) (at 353.7917 97.7106 0)
+      (effects (font (size 1.27 1.27)) (justify right) hide)
+    )
+  )
   (global_label "RXD" (shape output) (at 71.12 161.29 180) (fields_autoplaced)
     (effects (font (size 1.27 1.27)) (justify right))
@@
     )
   )
-  (global_label "FAN" (shape input) (at 382.27 125.73 0) (fields_autoplaced)
+  (global_label "BUZZER" (shape input) (at 382.27 125.73 0) (fields_autoplaced)
     (effects (font (size 1.27 1.27)) (justify left))
-    (property "Intersheet References" "${INTERSHEET_REFS}" (id 0) (at 388.1907 125.6506 0)
+    (property "Intersheet References" "${INTERSHEET_REFS}" (id 0) (at 392.1217 125.6506 0)
       (effects (font (size 1.27 1.27)) (justify left) hide)
     )
@@
     )
   )
-  (global_label "SCL" (shape input) (at 370.84 97.79 180) (fields_autoplaced)
-    (effects (font (size 1.27 1.27)) (justify right))
-    (property "Intersheet References" "${INTERSHEET_REFS}" (id 0) (at 364.9193 97.7106 0)
-      (effects (font (size 1.27 1.27)) (justify right) hide)
-    )
-  )
   (global_label "MENU" (shape output) (at 201.93 182.88 0) (fields_autoplaced)
     (effects (font (size 1.27 1.27)) (justify left))
@@
   (symbol (lib_id "HPS:GND") (at 370.84 104.14 0) (unit 1)
     (in_bom yes) (on_board yes) (fields_autoplaced)
-    (property "Reference" "#PWR?" (id 0) (at 370.84 110.49 0)
+    (property "Reference" "#PWR017" (id 0) (at 370.84 110.49 0)
       (effects (font (size 1.27 1.27)) hide)
     )
@@
     (pin "3")
   )
+  (symbol (lib_id "HPS:R_POT_10K") (at 311.15 43.18 90) (unit 1)
+    (in_bom yes) (on_board yes)
+    (property "Reference" "RV2" (id 0) (at 317.5 39.37 90))
+    (property "Value" "R_POT_10K" (id 1) (at 318.77 36.83 90))
+    (property "Footprint" "footprints:Potentiometer_Bourns_3386P_Vertical" (id 2) (at 322.58 43.18 0)
+      (effects (font (size 1.27 1.27)) hide)
+    )
+    (property "Datasheet" "https://www.bourns.com/docs/Product-Datasheets/3386.pdf" (id 3) (at 311.15 43.18 0)
+      (effects (font (size 1.27 1.27)) hide)
+    )
+    (property "MFG" "Bourns Inc." (id 4) (at 317.5 43.18 0)
+      (effects (font (size 1.27 1.27)) hide)
+    )
+    (property "MPN" "3386P-1-103TLF" (id 5) (at 320.04 43.18 0)
+      (effects (font (size 1.27 1.27)) hide)
+    )
+    (property "Digikey PN" "3386P-103TLF-ND" (id 6) (at 325.12 43.18 0)
+      (effects (font (size 1.27 1.27)) hide)
+    )
+    (property "Mouser PN" "N/A" (id 7) (at 327.66 43.18 0)
+      (effects (font (size 1.27 1.27)) hide)
+    )
+    (pin "1")
+    (pin "2")
+    (pin "3")
+  )
   (symbol (lib_id "HPS:C_0805_0.1uf") (at 63.5 166.37 90) (unit 1)
     (in_bom yes) (on_board yes)
@@
   (symbol (lib_id "HPS:VCC") (at 388.62 97.79 0) (unit 1)
     (in_bom yes) (on_board yes) (fields_autoplaced)
-    (property "Reference" "#PWR?" (id 0) (at 388.62 101.6 0)
+    (property "Reference" "#PWR019" (id 0) (at 388.62 101.6 0)
       (effects (font (size 1.27 1.27)) hide)
     )
@@
   )
   (symbol (lib_id "HPS:TC1602A-01T") (at 297.18 58.42 0) (unit 1)
-    (in_bom yes) (on_board yes) (fields_autoplaced)
+    (in_bom yes) (on_board yes)
     (property "Reference" "DS2" (id 0) (at 299.1994 35.56 0)
       (effects (font (size 1.27 1.27)) (justify left))
     )
-    (property "Value" "TC1602A-01T" (id 1) (at 299.1994 38.1 0)
+    (property "Value" "TC1602A-01T" (id 1) (at 299.72 33.02 0)
       (effects (font (size 1.27 1.27)) (justify left))
     )
@@
       (reference "#PWR016") (unit 1) (value "GND") (footprint "")
     )
+    (path "/067b45fc-db07-4f3a-9871-183fab03c716"
+      (reference "#PWR017") (unit 1) (value "GND") (footprint "")
+    )
     (path "/ed7cc89e-9495-4e2f-a9ca-3563ebdd30e8"
       (reference "#PWR018") (unit 1) (value "GND") (footprint "")
     )
+    (path "/3e0965fc-b789-493a-9f51-412a16a88e23"
+      (reference "#PWR019") (unit 1) (value "VCC") (footprint "")
+    )
     (path "/b3c36c95-a911-4edf-8a71-e8a00d2f2ff7"
       (reference "#PWR020") (unit 1) (value "VCC") (footprint "")
@@
       (reference "#PWR0104") (unit 1) (value "GND") (footprint "")
     )
-    (path "/067b45fc-db07-4f3a-9871-183fab03c716"
-      (reference "#PWR?") (unit 1) (value "GND") (footprint "")
-    )
-    (path "/3e0965fc-b789-493a-9f51-412a16a88e23"
-      (reference "#PWR?") (unit 1) (value "VCC") (footprint "")
-    )
     (path "/b625a70b-6b01-4ec2-b81a-d2af7627ba00"
       (reference "BT1") (unit 1) (value "Battery_Cell") (footprint "footprints:BatteryHolder_Keystone_106_1x20mm")
@@
       (reference "RV1") (unit 1) (value "R_POT_10K") (footprint "footprints:Potentiometer_Bourns_3386P_Vertical")
     )
+    (path "/0a8052d9-d064-4558-977d-840e6cd21b61"
+      (reference "RV2") (unit 1) (value "R_POT_10K") (footprint "footprints:Potentiometer_Bourns_3386P_Vertical")
+    )
     (path "/ccdcda96-f141-4ca2-9850-b5260a60df57"
