File: Gitclock/Gitclock.kicad_sch (KiCad schematic)
At the start: 42 parts, among them J1 PJ-102AH, J2 Conn_01x06, J3 Conn_01x05, SW1 Omron_B3F_SPST, SW2 Omron_B3F_SPST, SW3 Omron_B3F_SPST, SW4 Omron_B3F_SPST, SW5 RotaryEncoder_Switch, U1 ATmega328-PU, U2 L7805, U3 MAX7219, U4 DS1307_DIP-8, U5 ULN2003A, Y1 Crystal_16MHz, Y2 Crystal_32768Hz

Commit message: Gitclock
20220707
9:46AM
Parts:
- removed SW2: Omron_B3F_SPST, footprints:SW_SPST_Omron_B3FS-100xP, symbol HPS:Omron_B3F_SPST
- added R10, R12, R13, R7: R_0805_10K, footprints:R_0805_2012Metric, symbol HPS:R_0805_10K
Connections:
- net FAN is gone; now on net BUZZER: R11.2, SW4.1 (A), U1.15 (PB1)
- net BUZZER: now also U1.14 (PB0); no longer U1.12 (PD6)
- net GND: now also R10.2, R13.2, R7.2; no longer DS2.16 (LED(-)), SW5.B, U1.24 (PC1)
- net MENU: now also U1.25 (PC2); no longer U1.13 (PD7)
- net MENU OUTPUT2: now also U1.24 (PC1), R7.1; no longer U1.23 (PC0)
- net VCC: now also R12.2; no longer DS2.15 (LED(+))
- net SW2: now reaches U1.26 (PC3)
- net SW2: now also SW5.S2, R10.1
- net SNOOZE renamed MENU SCROLL
- net MENU SCROLL: now also SW5.B, U1.23 (PC0); no longer U1.14 (PB0)
- new net: DS2.15 (LED(+)), R12.1
- new net: DS2.16 (LED(-)), R13.1
- no-connect marks 37 -> 33
Other:
- note removed: "SNOOZE"
- moved on the sheet: BZ1, SW5

Commit message: 20220707Clock
12:22PM
Parts:
- removed R12, R13, R8, R9: R_0805_10K, footprints:R_0805_2012Metric, symbol HPS:R_0805_10K
- added C8, C9: C_0805_0.1uf, footprints:C_0805_2012Metric, symbol HPS:C_0805_0.1uf
- added R12: R_0805_47, footprints:R_0805_2012Metric, symbol HPS:R_0805_47
- added R13, R14: R_0805_1K, footprints:R_0805_2012Metric, symbol HPS:R_0805_1K
- added R8, R9: R_0805_4.7K, footprints:R_0805_2012Metric, symbol HPS:R_0805_4.7K
Connections:
- net BUZZER: now also U1.12 (PD6), U5.1 (I1); no longer R11.2, SW4.1 (A)
- net GND: now also C2.1, C7.1, DS2.2 (VDD), R2.1, RV1.1, RV1.3, SW3.1 (A), SW4.3 (B), SW5.S1, U1.20 (AVCC), U1.7 (VCC), U2.3 (OUT), U3.19 (V+), U4.8 (VCC), C8.1, C8.2, C9.1, C9.2, R13.2, R14.2, R8.1, R9.1
- net SCL: now also R9.2
- net SDA: now also R8.2
- net at DS1.10 (COM_DIG.3): now also U3.6 (DIG_2); no longer U3.7 (DIG_3)
- net at DS1.11 (COM_DIG.2): now also U3.11 (DIG_1); no longer U3.6 (DIG_2)
- net at DS1.14 (COM_DIG.1): now also U3.2 (DIG_0); no longer U3.11 (DIG_1)
- net at DS1.3 (DP), U3.22 (SEG_DP): now also DS1.8 (COLON)
- net at DS1.6 (COM_DIG.4): now also U3.7 (DIG_3); no longer U3.3 (DIG_4)
- net at DS1.7 (COM_COLON): now also U3.3 (DIG_4)
- net at DS2.15 (LED(+)): now also R13.1
- net at RV1.2: now also R12.1
- net at U3.18 (ISET): now also R12.2; no longer RV1.3
- net at DS2.16 (LED(-)): now also R14.1
- removed net VCC: C2.1, C7.1, DS2.2 (VDD), J3.2 (Pin_2), R2.1, RV1.1, SW3.1 (A), SW5.S1, U1.20 (AVCC), U1.7 (VCC), U2.3 (OUT), U3.19 (V+), U4.8 (VCC), U5.9 (COM)
- new net: J3.2 (Pin_2), U5.9 (COM)
- new net FAN_B: R11.2, SW4.1 (A)
- no-connect marks 33 -> 31
Other:
- note added: "FAN Button"
- moved on the sheet: DS1, J3, R11, RV1, SW4, U5

Commit message: Latest: 20220707
12:32PM Gitclock Update
Connections:
- net BUZZER: now also U1.13 (PD7); no longer U1.12 (PD6), U1.14 (PB0), U1.15 (PB1), U5.1 (I1)
- net FAN_B: now also U1.17 (PB3)
- net MOSI: no longer U1.17 (PB3), U3.1 (DIN)
- net SCK renamed LED_SCK
- net LED_SCK: no longer U3.13 (CLK)
- net SS renamed DATA
- net DATA: now also U3.1 (DIN); no longer U3.12 (LOAD)
- new net CLK: U1.15 (PB1), U3.13 (CLK)
- new net FAN: U1.12 (PD6), U5.1 (I1)
- new net LOAD: U1.14 (PB0), U3.12 (LOAD)
- no-connect marks 31 -> 30
Changed lines of the file:
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@@
   (no_connect (at 304.8 127))
   (no_connect (at 304.8 119.38))
-  (no_connect (at 198.12 182.88))
   (no_connect (at 287.02 55.88))
   (no_connect (at 287.02 60.96))
@@
     (stroke (width 0) (type default) (color 0 0 0 0))
   )
+  (wire (pts (xy 198.12 127) (xy 199.39 127))
+    (stroke (width 0) (type default) (color 0 0 0 0))
+  )
   (polyline (pts (xy 407.67 85.09) (xy 334.01 85.09))
     (stroke (width 0) (type default) (color 0 0 0 0))
@@
     (stroke (width 0) (type default) (color 0 0 0 0))
   )
-  (wire (pts (xy 198.12 127) (xy 201.93 127))
-    (stroke (width 0) (type default) (color 0 0 0 0))
-  )
   (polyline (pts (xy 133.35 85.09) (xy 133.35 12.7))
     (stroke (width 0) (type default) (color 0 0 0 0))
@@
     (stroke (width 0) (type default) (color 0 0 0 0))
   )
+  (wire (pts (xy 198.12 121.92) (xy 199.39 121.92))
+    (stroke (width 0) (type default) (color 0 0 0 0))
+  )
   (wire (pts (xy 52.07 60.96) (xy 118.11 60.96))
     (stroke (width 0) (type default) (color 0 0 0 0))
@@
     (stroke (width 0) (type default) (color 0 0 0 0))
   )
-  (wire (pts (xy 198.12 129.54) (xy 203.2 129.54))
-    (stroke (width 0) (type default) (color 0 0 0 0))
-  )
   (wire (pts (xy 27.94 68.58) (xy 31.75 68.58))
     (stroke (width 0) (type default) (color 0 0 0 0))
@@
     (stroke (width 0) (type default) (color 0 0 0 0))
   )
-  (wire (pts (xy 198.12 124.46) (xy 198.12 121.92))
-    (stroke (width 0) (type default) (color 0 0 0 0))
-  )
   (wire (pts (xy 52.07 50.8) (xy 74.93 50.8))
     (stroke (width 0) (type default) (color 0 0 0 0))
@@
   )
   (polyline (pts (xy 265.43 97.79) (xy 265.43 99.06))
+    (stroke (width 0) (type default) (color 0 0 0 0))
+  )
+  (wire (pts (xy 198.12 124.46) (xy 199.39 124.46))
     (stroke (width 0) (type default) (color 0 0 0 0))
   )
@@
     (effects (font (size 3 3)) (justify left bottom))
   )
-  (global_label "FAN" (shape output) (at 198.12 124.46 0) (fields_autoplaced)
-    (effects (font (size 1.27 1.27)) (justify left))
-    (property "Intersheet References" "${INTERSHEET_REFS}" (id 0) (at 204.0407 124.3806 0)
-      (effects (font (size 1.27 1.27)) (justify left) hide)
+  (global_label "FAN_B" (shape output) (at 198.12 129.54 0) (fields_autoplaced)
+    (effects (font (size 1.27 1.27)) (justify left))
+    (property "Intersheet References" "${INTERSHEET_REFS}" (id 0) (at 206.2783 129.4606 0)
+      (effects (font (size 1.27 1.27)) (justify left) hide)
+    )
+  )
+  (global_label "CLK" (shape input) (at 27.94 68.58 180) (fields_autoplaced)
+    (effects (font (size 1.27 1.27)) (justify right))
+    (property "Intersheet References" "${INTERSHEET_REFS}" (id 0) (at 21.9588 68.5006 0)
+      (effects (font (size 1.27 1.27)) (justify right) hide)
     )
   )
@@
     )
   )
-  (global_label "SCK" (shape output) (at 200.66 134.62 0) (fields_autoplaced)
-    (effects (font (size 1.27 1.27)) (justify left))
-    (property "Intersheet References" "${INTERSHEET_REFS}" (id 0) (at 206.8226 134.5406 0)
-      (effects (font (size 1.27 1.27)) (justify left) hide)
-    )
-  )
-  (global_label "MOSI" (shape output) (at 203.2 129.54 0) (fields_autoplaced)
-    (effects (font (size 1.27 1.27)) (justify left))
-    (property "Intersheet References" "${INTERSHEET_REFS}" (id 0) (at 210.2093 129.4606 0)
+  (global_label "LED_SCK" (shape output) (at 200.66 134.62 0) (fields_autoplaced)
+    (effects (font (size 1.27 1.27)) (justify left))
+    (property "Intersheet References" "${INTERSHEET_REFS}" (id 0) (at 211.2374 134.5406 0)
+      (effects (font (size 1.27 1.27)) (justify left) hide)
+    )
+  )
+  (global_label "DATA" (shape output) (at 199.39 127 0) (fields_autoplaced)
+    (effects (font (size 1.27 1.27)) (justify left))
+    (property "Intersheet References" "${INTERSHEET_REFS}" (id 0) (at 206.2179 126.9206 0)
       (effects (font (size 1.27 1.27)) (justify left) hide)
     )
@@
     )
   )
-  (global_label "SS" (shape output) (at 201.93 127 0) (fields_autoplaced)
-    (effects (font (size 1.27 1.27)) (justify left))
-    (property "Intersheet References" "${INTERSHEET_REFS}" (id 0) (at 206.7621 126.9206 0)
+  (global_label "LOAD" (shape output) (at 199.39 121.92 0) (fields_autoplaced)
+    (effects (font (size 1.27 1.27)) (justify left))
+    (property "Intersheet References" "${INTERSHEET_REFS}" (id 0) (at 206.5202 121.8406 0)
       (effects (font (size 1.27 1.27)) (justify left) hide)
     )
@@
     )
   )
-  (global_label "SS" (shape input) (at 29.21 66.04 180) (fields_autoplaced)
-    (effects (font (size 1.27 1.27)) (justify right))
-    (property "Intersheet References" "${INTERSHEET_REFS}" (id 0) (at 24.3779 65.9606 0)
-      (effects (font (size 1.27 1.27)) (justify right) hide)
-    )
-  )
-  (global_label "SCK" (shape input) (at 27.94 68.58 180) (fields_autoplaced)
-    (effects (font (size 1.27 1.27)) (justify right))
-    (property "Intersheet References" "${INTERSHEET_REFS}" (id 0) (at 21.7774 68.5006 0)
+  (global_label "LOAD" (shape input) (at 29.21 66.04 180) (fields_autoplaced)
+    (effects (font (size 1.27 1.27)) (justify right))
+    (property "Intersheet References" "${INTERSHEET_REFS}" (id 0) (at 22.0798 65.9606 0)
       (effects (font (size 1.27 1.27)) (justify right) hide)
     )
@@
     )
   )
-  (global_label "BUZZER" (shape output) (at 198.12 121.92 0) (fields_autoplaced)
-    (effects (font (size 1.27 1.27)) (justify left))
-    (property "Intersheet References" "${INTERSHEET_REFS}" (id 0) (at 207.9717 121.8406 0)
-      (effects (font (size 1.27 1.27)) (justify left) hide)
-    )
-  )
-  (global_label "SCK" (shape input) (at 118.11 107.95 90) (fields_autoplaced)
-    (effects (font (size 1.27 1.27)) (justify left))
-    (property "Intersheet References" "${INTERSHEET_REFS}" (id 0) (at 118.0306 101.7874 90)
+  (global_label "BUZZER" (shape output) (at 198.12 182.88 0) (fields_autoplaced)
+    (effects (font (size 1.27 1.27)) (justify left))
+    (property "Intersheet References" "${INTERSHEET_REFS}" (id 0) (at 207.9717 182.8006 0)
+      (effects (font (size 1.27 1.27)) (justify left) hide)
+    )
+  )
+  (global_label "LED_SCK" (shape input) (at 118.11 107.95 90) (fields_autoplaced)
+    (effects (font (size 1.27 1.27)) (justify left))
+    (property "Intersheet References" "${INTERSHEET_REFS}" (id 0) (at 118.0306 97.3726 90)
+      (effects (font (size 1.27 1.27)) (justify left) hide)
+    )
+  )
+  (global_label "CLK" (shape output) (at 199.39 124.46 0) (fields_autoplaced)
+    (effects (font (size 1.27 1.27)) (justify left))
+    (property "Intersheet References" "${INTERSHEET_REFS}" (id 0) (at 205.3712 124.3806 0)
       (effects (font (size 1.27 1.27)) (justify left) hide)
     )
@@
     )
   )
-  (global_label "MOSI" (shape input) (at 29.21 71.12 180) (fields_autoplaced)
-    (effects (font (size 1.27 1.27)) (justify right))
-    (property "Intersheet References" "${INTERSHEET_REFS}" (id 0) (at 22.2007 71.0406 0)
-      (effects (font (size 1.27 1.27)) (justify right) hide)
-    )
+  (global_label "DATA" (shape input) (at 29.21 71.12 180) (fields_autoplaced)
+    (effects (font (size 1.27 1.27)) (justify right))
+    (property "Intersheet References" "${INTERSHEET_REFS}" (id 0) (at 22.3821 71.0406 0)
+      (effects (font (size 1.27 1.27)) (justify right) hide)
+    )

Commit message: Gitclock
20220707
1:15PM
Parts:
- removed R12: R_0805_47, footprints:R_0805_2012Metric, symbol HPS:R_0805_47
- removed R13, R14: R_0805_1K, footprints:R_0805_2012Metric, symbol HPS:R_0805_1K
- added R12: R_0805_10K, footprints:R_0805_2012Metric, symbol HPS:R_0805_10K
- added R?: R_0805_47, footprints:R_0805_2012Metric, symbol HPS:R_0805_47
Connections:
- net FAN: now also R11.2, SW4.1 (A); no longer U5.1 (I1)
- net GND: now also DS2.16 (LED(-)), RV2.1, RV2.3, R12.2, R?.2; no longer RV1.1, RV1.3, SW4.3 (B)
- net MOSI: now also U1.17 (PB3)
- net at DS2.3 (VO): now also RV2.2; no longer RV2.1
- net at SW4.4 (B): now also U5.2 (I2)
- net at RV1.2: now also RV1.1, R12.1
- net at U3.18 (ISET): now also RV1.3
- net at DS2.15 (LED(+)): now also R?.1
- removed net FAN_B: R11.2, SW4.1 (A), U1.17 (PB3)
- new net: SW4.3 (B), U5.1 (I1)
- no-connect marks 30 -> 29
Other:
- note added: "Mechanical"
- note removed: "FAN Button"
- moved on the sheet: H2, H3, H4, R11, RV2, SW4

Commit message: Gitclock
20220707
3:55PM
Parts:
- removed R11: R_0805_10K, footprints:R_0805_2012Metric, symbol HPS:R_0805_10K
- removed SW4: Omron_B3F_SPST, footprints:SW_SPST_Omron_B3FS-100xP, symbol HPS:Omron_B3F_SPST
- gave numbers to parts that had none: 1
Connections:
- net FAN: now also U5.1 (I1)
- net MENU renamed FAN_B
- net SW2 renamed MENU_B
- no-connect marks 29 -> 28
Changed lines of the file:
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@@
   (junction (at 392.43 69.85) (diameter 0) (color 0 0 0 0)
   )
-  (junction (at 289.56 118.11) (diameter 0) (color 0 0 0 0)
-  )
   (junction (at 50.8 166.37) (diameter 0) (color 0 0 0 0)
   )
@@
   (no_connect (at 38.1 118.11))
   (no_connect (at 304.8 129.54))
-  (no_connect (at 294.64 119.38))
   (no_connect (at -44.45 233.68))
   (no_connect (at 377.19 27.94))
@@
     (stroke (width 0) (type default) (color 0 0 0 0))
   )
-  (wire (pts (xy 287.02 118.11) (xy 289.56 118.11))
-    (stroke (width 0) (type default) (color 0 0 0 0))
-  )
   (polyline (pts (xy 12.7 256.54) (xy 53.34 256.54))
     (stroke (width 0) (type default) (color 0 0 0 0))
@@
     (stroke (width 0) (type default) (color 0 0 0 0))
   )
-  (wire (pts (xy 289.56 118.11) (xy 294.64 118.11))
-    (stroke (width 0) (type default) (color 0 0 0 0))
-  )
   (wire (pts (xy 125.73 24.13) (xy 125.73 35.56))
     (stroke (width 0) (type default) (color 0 0 0 0))
@@
     (stroke (width 0) (type default) (color 0 0 0 0))
   )
-  (wire (pts (xy 294.64 118.11) (xy 294.64 116.84))
-    (stroke (width 0) (type default) (color 0 0 0 0))
-  )
   (wire (pts (xy 368.3 55.88) (xy 368.3 64.77))
     (stroke (width 0) (type default) (color 0 0 0 0))
@@
     )
   )
-  (global_label "SW2" (shape output) (at 198.12 152.4 0) (fields_autoplaced)
+  (global_label "MENU_B" (shape output) (at 198.12 152.4 0) (fields_autoplaced)
     (effects (font (size 1.27 1.27)) (justify left))
-    (property "Intersheet References" "${INTERSHEET_REFS}" (id 0) (at 204.4036 152.3206 0)
+    (property "Intersheet References" "${INTERSHEET_REFS}" (id 0) (at 208.0321 152.3206 0)
       (effects (font (size 1.27 1.27)) (justify left) hide)
     )
@@
     )
   )
-  (global_label "MENU" (shape input) (at 370.84 30.48 180) (fields_autoplaced)
+  (global_label "FAN_B" (shape input) (at 370.84 30.48 180) (fields_autoplaced)
     (effects (font (size 1.27 1.27)) (justify right))
-    (property "Intersheet References" "${INTERSHEET_REFS}" (id 0) (at 363.1655 30.4006 0)
+    (property "Intersheet References" "${INTERSHEET_REFS}" (id 0) (at 362.6817 30.4006 0)
       (effects (font (size 1.27 1.27)) (justify right) hide)
     )
@@
     )
   )
-  (global_label "FAN" (shape input) (at 287.02 118.11 180) (fields_autoplaced)
+  (global_label "FAN" (shape input) (at 304.8 116.84 180) (fields_autoplaced)
     (effects (font (size 1.27 1.27)) (justify right))
-    (property "Intersheet References" "${INTERSHEET_REFS}" (id 0) (at 281.0993 118.0306 0)
+    (property "Intersheet References" "${INTERSHEET_REFS}" (id 0) (at 298.8793 116.7606 0)
       (effects (font (size 1.27 1.27)) (justify right) hide)
     )
@@
     )
   )
-  (global_label "SW2" (shape input) (at 394.97 69.85 0) (fields_autoplaced)
+  (global_label "MENU_B" (shape input) (at 394.97 69.85 0) (fields_autoplaced)
     (effects (font (size 1.27 1.27)) (justify left))
-    (property "Intersheet References" "${INTERSHEET_REFS}" (id 0) (at 401.2536 69.7706 0)
+    (property "Intersheet References" "${INTERSHEET_REFS}" (id 0) (at 404.8821 69.7706 0)
       (effects (font (size 1.27 1.27)) (justify left) hide)
     )
@@
     )
   )
-  (global_label "MENU" (shape output) (at 198.12 149.86 0) (fields_autoplaced)
+  (global_label "FAN_B" (shape output) (at 198.12 149.86 0) (fields_autoplaced)
     (effects (font (size 1.27 1.27)) (justify left))
-    (property "Intersheet References" "${INTERSHEET_REFS}" (id 0) (at 205.7945 149.7806 0)
+    (property "Intersheet References" "${INTERSHEET_REFS}" (id 0) (at 206.2783 149.7806 0)
       (effects (font (size 1.27 1.27)) (justify left) hide)
     )
@@
     (pin "2")
   )
-  (symbol (lib_id "HPS:R_0805_10K") (at 289.56 121.92 180) (unit 1)
-    (in_bom yes) (on_board yes)
-    (property "Reference" "R11" (id 0) (at 295.91 124.46 0)
-      (effects (font (size 1.27 1.27)) (justify left))
-    )
-    (property "Value" "R_0805_10K" (id 1) (at 303.53 121.92 0)
-      (effects (font (size 1.27 1.27)) (justify left))
-    )
-    (property "Footprint" "footprints:R_0805_2012Metric" (id 2) (at 289.56 105.41 0)
-      (effects (font (size 1.27 1.27)) hide)
-    )
-    (property "Datasheet" "https://www.digikey.com/en/products/detail/yageo/RC0805FR-0710KL/727535" (id 3) (at 292.1 121.92 0)
-      (effects (font (size 1.27 1.27)) hide)
-    )
-    (property "MFG" "Yageo" (id 4) (at 289.56 110.49 0)
-      (effects (font (size 1.27 1.27)) hide)
-    )
-    (property "MPN" "RC0805FR-0710KL" (id 5) (at 289.56 107.95 0)
-      (effects (font (size 1.27 1.27)) hide)
-    )
-    (property "Digikey PN" "311-10.0KCRCT-ND" (id 6) (at 289.56 102.87 0)
-      (effects (font (size 1.27 1.27)) hide)
-    )
-    (property "Mouser PN" "N/A" (id 7) (at 289.56 100.33 0)
-      (effects (font (size 1.27 1.27)) hide)
-    )
-    (property "Power" "N/A" (id 8) (at 289.56 97.79 0)
-      (effects (font (size 1.27 1.27)) hide)
-    )
-    (property "Tolerance" "N/A" (id 9) (at 289.56 95.25 0)
-      (effects (font (size 1.27 1.27)) hide)
-    )
-    (pin "1")
-    (pin "2")
-  )
   (symbol (lib_id "HPS:GND") (at 158.75 50.8 0) (unit 1)
     (in_bom yes) (on_board yes) (fields_autoplaced)
@@
   (symbol (lib_id "HPS:R_0805_47") (at 311.15 50.8 90) (unit 1)
     (in_bom yes) (on_board yes)
-    (property "Reference" "R?" (id 0) (at 311.15 45.72 90))
+    (property "Reference" "R13" (id 0) (at 311.15 45.72 90))
     (property "Value" "R_0805_47" (id 1) (at 311.15 46.99 90))
     (property "Footprint" "footprints:R_0805_2012Metric" (id 2) (at 327.66 50.8 0)
@@
     (pin "2")
   )
-  (symbol (lib_id "HPS:Omron_B3F_SPST") (at 299.72 116.84 0) (unit 1)
-    (in_bom yes) (on_board yes)
-    (property "Reference" "SW4" (id 0) (at 299.72 111.76 0))
-    (property "Value" "Omron_B3F_SPST" (id 1) (at 300.99 113.03 0))
-    (property "Footprint" "footprints:SW_SPST_Omron_B3FS-100xP" (id 2) (at 299.72 128.27 0)
-      (effects (font (size 1.27 1.27)) hide)
-    )
-    (property "Datasheet" "https://omronfs.omron.com/en_US/ecb/products/pdf/en-b3fs.pdf" (id 3) (at 299.72 116.84 0)
-      (effects (font (size 1.27 1.27)) hide)
-    )
-    (property "MFG" "Omron Electronics Inc-EMC Div" (id 4) (at 299.72 123.19 0)
-      (effects (font (size 1.27 1.27)) hide)
-    )
-    (property "MPN" "B3FS-1000P" (id 5) (at 299.72 125.73 0)
-      (effects (font (size 1.27 1.27)) hide)
-    )
-    (property "Digikey PN" "SW423CT-ND" (id 6) (at 299.72 130.81 0)
-      (effects (font (size 1.27 1.27)) hide)
-    )
-    (property "Mouser PN" "N/A" (id 7) (at 299.72 133.35 0)
-      (effects (font (size 1.27 1.27)) hide)
-    )
-    (pin "1")
-    (pin "2")
-    (pin "3")
-    (pin "4")
-  )
   (symbol (lib_id "HPS:Conn_01x05") (at 351.79 114.3 0) (unit 1)
     (in_bom yes) (on_board yes) (fields_autoplaced)
@@
     (pin "1")
   )
-  (symbol (lib_id "HPS:GND") (at 289.56 125.73 0) (unit 1)
-    (in_bom yes) (on_board yes) (fields_autoplaced)
-    (property "Reference" "#PWR026" (id 0) (at 289.56 132.08 0)
-      (effects (font (size 1.27 1.27)) hide)
-    )
-    (property "Value" "GND" (id 1) (at 289.56 130.81 0))
-    (property "Footprint" "" (id 2) (at 289.56 125.73 0)
-      (effects (font (size 1.27 1.27)) hide)
-    )
-    (property "Datasheet" "" (id 3) (at 289.56 125.73 0)
-      (effects (font (size 1.27 1.27)) hide)
-    )
-    (pin "1")
-  )
   (symbol (lib_id "HPS:VCC") (at 226.06 157.48 0) (unit 1)
     (in_bom yes) (on_board yes) (fields_autoplaced)
@@
       (reference "#PWR025") (unit 1) (value "VCC") (footprint "")
     )
-    (path "/b2f7aa7c-1b8a-4b2a-b447-22be93212478"
-      (reference "#PWR026") (unit 1) (value "GND") (footprint "")
-    )
     (path "/8c65d00e-4e5a-48ab-a9c0-5de3e6fe5922"
       (reference "#PWR027") (unit 1) (value "GND") (footprint "")
@@
       (reference "R10") (unit 1) (value "R_0805_10K") (footprint "footprints:R_0805_2012Metric")
     )
-    (path "/17ccefeb-a492-427b-8efd-13f0e4786ae3"
-      (reference "R11") (unit 1) (value "R_0805_10K") (footprint "footprints:R_0805_2012Metric")
-    )
     (path "/b0f86ab7-7df7-4c72-b3df-3ad8d1387d04"
       (reference "R12") (unit 1) (value "R_0805_10K") (footprint "footprints:R_0805_2012Metric")
     )
     (path "/2ca21dc6-a94f-4c50-8937-3d67d5067a4f"
-      (reference "R?") (unit 1) (value "R_0805_47") (footprint "footprints:R_0805_2012Metric")
+      (reference "R13") (unit 1) (value "R_0805_47") (footprint "footprints:R_0805_2012Metric")
     )
     (path "/99c06508-6a16-489f-a186-ced706cf79b5"
@@
       (reference "SW3") (unit 1) (value "Omron_B3F_SPST") (footprint "footprints:SW_SPST_Omron_B3FS-100xP")
     )
-    (path "/5f30d32f-818b-4e3a-9a53-1ff51ebb71a9"
-      (reference "SW4") (unit 1) (value "Omron_B3F_SPST") (footprint "footprints:SW_SPST_Omron_B3FS-100xP")
-    )
     (path "/9f3718d2-4c44-41a2-bdc9-fa0fdcd56d8e"

Commit message: 20220713
5:40 PM clock
Parts:
- removed J3: Conn_01x05, footprints:PinHeader_1x05_P2.54mm_Vertical, symbol HPS:Conn_01x05
- removed U5: ULN2003A, footprints:DIP-16_W7.62mm, symbol HPS:ULN2003A
Connections:
- net GND: no longer C2.1, C7.1, C8.1, C9.1, DS2.2 (VDD), R12.2, R13.2, R2.1, R8.1, R9.1, RV2.3, SW3.1 (A), SW5.S1, U1.20 (AVCC), U1.7 (VCC), U2.3 (OUT), U3.19 (V+), U4.8 (VCC)
- net FAN: no longer names the net of U1.12 (PD6)
- net FAN_B renamed Select_B
- new net VCC: C2.1, C7.1, C8.1, C9.1, DS2.2 (VDD), R12.2, R13.2, R2.1, R8.1, R9.1, RV2.3, SW3.1 (A), SW5.S1, U1.20 (AVCC), U1.7 (VCC), U2.3 (OUT), U3.19 (V+), U4.8 (VCC)
- no-connect marks 28 -> 15
Other:
- note added: "Select Button"
- note removed: "FAN"
- note removed: "MENU"
- moved on the sheet: BZ1, DS2, R10, R13, R6, R7, RV2, SW5

Commit message: Routing display
Parts:
- U2: footprint (none) -> footprints:TO-252-2; Digikey PN (none) -> 497-7255-1-ND; MFG (none) -> STMicroelectronics; MPN (none) -> L7805CDT-TR
Changed lines of the file:
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@@
     (property "Reference" "U2" (id 0) (at 73.66 106.68 0))
     (property "Value" "L7805" (id 1) (at 73.66 109.22 0))
-    (property "Footprint" "" (id 2) (at 74.295 118.11 0)
+    (property "Footprint" "footprints:TO-252-2" (id 2) (at 74.295 118.11 0)
       (effects (font (size 1.27 1.27) italic) (justify left) hide)
     )
     (property "Datasheet" "http://www.st.com/content/ccc/resource/technical/document/datasheet/41/4f/b3/b0/12/d4/47/88/CD00000444.pdf/files/CD00000444.pdf/jcr:content/translations/en.CD00000444.pdf" (id 3) (at 73.66 115.57 0)
+      (effects (font (size 1.27 1.27)) hide)
+    )
+    (property "Digikey PN" "497-7255-1-ND" (id 4) (at 73.66 114.3 0)
+      (effects (font (size 1.27 1.27)) hide)
+    )
+    (property "MPN" "L7805CDT-TR" (id 5) (at 73.66 114.3 0)
+      (effects (font (size 1.27 1.27)) hide)
+    )
+    (property "MFG" "STMicroelectronics" (id 6) (at 73.66 114.3 0)
       (effects (font (size 1.27 1.27)) hide)
     )
@@
     )
     (path "/b0091a18-5817-4636-b5cf-c91a780fd88c"
-      (reference "U2") (unit 1) (value "L7805") (footprint "")
+      (reference "U2") (unit 1) (value "L7805") (footprint "footprints:TO-252-2")
     )
     (path "/f3d9e45b-157d-42f3-bf90-97a41295fbdc"
