File: Gitclock/Gitclock.kicad_sch (KiCad schematic)
At the start: 43 parts, among them J1 PJ-102AH, J2 Conn_01x06, SW1 Omron_B3F_SPST, SW3 Omron_B3F_SPST, SW5 RotaryEncoder_Switch, U1 ATmega328-PU, U2 L7805, U3 MAX7219, U4 DS1307_DIP-8, Y1 Crystal_16MHz, Y2 Crystal_32768Hz

Commit message: Final Routing Pass
Parts:
- removed R5: R_0805_10K, footprints:R_0805_2012Metric, symbol HPS:R_0805_10K
- removed SW3: Omron_B3F_SPST, footprints:SW_SPST_Omron_B3FS-100xP, symbol HPS:Omron_B3F_SPST
Connections:
- no-connect marks 15 -> 13
Other:
- note removed: "Select Button"
Changed lines of the file:
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@@
   (junction (at 68.58 45.72) (diameter 0) (color 0 0 0 0)
   )
-  (junction (at 373.38 30.48) (diameter 0) (color 0 0 0 0)
-  )
   (junction (at 182.88 193.04) (diameter 0) (color 0 0 0 0)
   )
@@
   (no_connect (at 38.1 118.11))
   (no_connect (at -44.45 233.68))
-  (no_connect (at 377.19 27.94))
-  (no_connect (at 387.35 27.94))
   (no_connect (at 213.36 60.96))
   (wire (pts (xy 68.58 45.72) (xy 68.58 17.78))
@@
     (stroke (width 0) (type default) (color 0 0 0 0))
   )
-  (polyline (pts (xy 358.14 20.32) (xy 358.14 19.05))
-    (stroke (width 0) (type default) (color 0 0 0 0))
-  )
   (wire (pts (xy 41.91 80.01) (xy 41.91 81.28))
     (stroke (width 0) (type default) (color 0 0 0 0))
@@
     (stroke (width 0) (type default) (color 0 0 0 0))
   )
-  (polyline (pts (xy 400.05 21.59) (xy 400.05 46.99))
-    (stroke (width 0) (type default) (color 0 0 0 0))
-  )
   (wire (pts (xy 20.32 22.86) (xy 24.13 22.86))
     (stroke (width 0) (type default) (color 0 0 0 0))
@@
     (stroke (width 0) (type default) (color 0 0 0 0))
   )
-  (wire (pts (xy 370.84 30.48) (xy 373.38 30.48))
-    (stroke (width 0) (type default) (color 0 0 0 0))
-  )
   (wire (pts (xy 361.95 71.12) (xy 361.95 66.04))
     (stroke (width 0) (type default) (color 0 0 0 0))
@@
     (stroke (width 0) (type default) (color 0 0 0 0))
   )
-  (polyline (pts (xy 356.87 21.59) (xy 358.14 20.32))
-    (stroke (width 0) (type default) (color 0 0 0 0))
-  )
   (wire (pts (xy 213.36 139.7) (xy 213.36 142.24))
     (stroke (width 0) (type default) (color 0 0 0 0))
@@
     (stroke (width 0) (type default) (color 0 0 0 0))
   )
-  (wire (pts (xy 391.16 30.48) (xy 387.35 30.48))
-    (stroke (width 0) (type default) (color 0 0 0 0))
-  )
   (wire (pts (xy 219.71 134.62) (xy 232.41 134.62))
     (stroke (width 0) (type default) (color 0 0 0 0))
@@
     (stroke (width 0) (type default) (color 0 0 0 0))
   )
-  (wire (pts (xy 373.38 30.48) (xy 377.19 30.48))
-    (stroke (width 0) (type default) (color 0 0 0 0))
-  )
   (wire (pts (xy 259.08 134.62) (xy 259.08 142.24))
     (stroke (width 0) (type default) (color 0 0 0 0))
   )
-  (polyline (pts (xy 356.87 21.59) (xy 400.05 21.59))
-    (stroke (width 0) (type default) (color 0 0 0 0))
-  )
   (polyline (pts (xy 234.95 86.36) (xy 234.95 20.32))
     (stroke (width 0) (type default) (color 0 0 0 0))
@@
     (stroke (width 0) (type default) (color 0 0 0 0))
   )
-  (polyline (pts (xy 356.87 46.99) (xy 356.87 21.59))
-    (stroke (width 0) (type default) (color 0 0 0 0))
-  )
-  (polyline (pts (xy 400.05 46.99) (xy 356.87 46.99))
-    (stroke (width 0) (type default) (color 0 0 0 0))
-  )
   (polyline (pts (xy 16.51 12.7) (xy 16.51 19.05))
     (stroke (width 0) (type default) (color 0 0 0 0))
@@
     (effects (font (size 1.27 1.27)) (justify left bottom))
   )
-  (text "Select Button\n" (at 358.14 25.4 0)
-    (effects (font (size 1.27 1.27)) (justify left bottom))
-  )
   (text "Mechanical" (at 13.97 259.08 0)
     (effects (font (size 1.27 1.27)) (justify left bottom))
@@
     )
   )
-  (global_label "Select_B" (shape input) (at 370.84 30.48 180) (fields_autoplaced)
-    (effects (font (size 1.27 1.27)) (justify right))
-    (property "Intersheet References" "${INTERSHEET_REFS}" (id 0) (at 360.3231 30.4006 0)
-      (effects (font (size 1.27 1.27)) (justify right) hide)
-    )
-  )
   (global_label "D6" (shape bidirectional) (at 198.12 175.26 0) (fields_autoplaced)
     (effects (font (size 1.27 1.27)) (justify left))
@@
     (pin "2")
   )
-  (symbol (lib_id "HPS:R_0805_10K") (at 373.38 34.29 180) (unit 1)
-    (in_bom yes) (on_board yes)
-    (property "Reference" "R5" (id 0) (at 365.76 35.56 0)
-      (effects (font (size 1.27 1.27)) (justify left))
-    )
-    (property "Value" "R_0805_10K" (id 1) (at 370.84 33.0201 0)
-      (effects (font (size 1.27 1.27)) (justify left))
-    )
-    (property "Footprint" "footprints:R_0805_2012Metric" (id 2) (at 373.38 17.78 0)
-      (effects (font (size 1.27 1.27)) hide)
-    )
-    (property "Datasheet" "https://www.digikey.com/en/products/detail/yageo/RC0805FR-0710KL/727535" (id 3) (at 375.92 34.29 0)
-      (effects (font (size 1.27 1.27)) hide)
-    )
-    (property "MFG" "Yageo" (id 4) (at 373.38 22.86 0)
-      (effects (font (size 1.27 1.27)) hide)
-    )
-    (property "MPN" "RC0805FR-0710KL" (id 5) (at 373.38 20.32 0)
-      (effects (font (size 1.27 1.27)) hide)
-    )
-    (property "Digikey PN" "311-10.0KCRCT-ND" (id 6) (at 373.38 15.24 0)
-      (effects (font (size 1.27 1.27)) hide)
-    )
-    (property "Mouser PN" "N/A" (id 7) (at 373.38 12.7 0)
-      (effects (font (size 1.27 1.27)) hide)
-    )
-    (property "Power" "N/A" (id 8) (at 373.38 10.16 0)
-      (effects (font (size 1.27 1.27)) hide)
-    )
-    (property "Tolerance" "N/A" (id 9) (at 373.38 7.62 0)
-      (effects (font (size 1.27 1.27)) hide)
-    )
-    (pin "1")
-    (pin "2")
-  )
   (symbol (lib_id "HPS:GND") (at 182.88 195.58 0) (unit 1)
     (in_bom yes) (on_board yes) (fields_autoplaced)
@@
     (pin "1")
   )
-  (symbol (lib_id "HPS:VCC") (at 391.16 30.48 0) (unit 1)
-    (in_bom yes) (on_board yes) (fields_autoplaced)
-    (property "Reference" "#PWR011" (id 0) (at 391.16 34.29 0)
-      (effects (font (size 1.27 1.27)) hide)
-    )
-    (property "Value" "VCC" (id 1) (at 391.16 25.4 0))
-    (property "Footprint" "" (id 2) (at 391.16 30.48 0)
-      (effects (font (size 1.27 1.27)) hide)
-    )
-    (property "Datasheet" "" (id 3) (at 391.16 30.48 0)
-      (effects (font (size 1.27 1.27)) hide)
-    )
-    (pin "1")
-  )
   (symbol (lib_id "HPS:GND") (at 259.08 152.4 0) (unit 1)
     (in_bom yes) (on_board yes) (fields_autoplaced)
@@
     (pin "2")
   )
-  (symbol (lib_id "HPS:GND") (at 373.38 38.1 0) (unit 1)
-    (in_bom yes) (on_board yes)
-    (property "Reference" "#PWR012" (id 0) (at 373.38 44.45 0)
-      (effects (font (size 1.27 1.27)) hide)
-    )
-    (property "Value" "GND" (id 1) (at 373.38 43.18 0))
-    (property "Footprint" "" (id 2) (at 373.38 38.1 0)
-      (effects (font (size 1.27 1.27)) hide)
-    )
-    (property "Datasheet" "" (id 3) (at 373.38 38.1 0)
-      (effects (font (size 1.27 1.27)) hide)
-    )
-    (pin "1")
-  )
   (symbol (lib_id "HPS:MAX7219") (at 41.91 50.8 0) (unit 1)
     (in_bom yes) (on_board yes) (fields_autoplaced)
@@
     (pin "1")
   )
-  (symbol (lib_id "HPS:Omron_B3F_SPST") (at 382.27 30.48 180) (unit 1)
-    (in_bom yes) (on_board yes)
-    (property "Reference" "SW3" (id 0) (at 382.27 36.83 0))
-    (property "Value" "Omron_B3F_SPST" (id 1) (at 382.27 39.37 0))
-    (property "Footprint" "footprints:SW_SPST_Omron_B3FS-100xP" (id 2) (at 382.27 19.05 0)
-      (effects (font (size 1.27 1.27)) hide)
-    )
-    (property "Datasheet" "https://omronfs.omron.com/en_US/ecb/products/pdf/en-b3fs.pdf" (id 3) (at 382.27 30.48 0)
-      (effects (font (size 1.27 1.27)) hide)
-    )
-    (property "MFG" "Omron Electronics Inc-EMC Div" (id 4) (at 382.27 24.13 0)
-      (effects (font (size 1.27 1.27)) hide)
-    )
-    (property "MPN" "B3FS-1000P" (id 5) (at 382.27 21.59 0)
-      (effects (font (size 1.27 1.27)) hide)
-    )
-    (property "Digikey PN" "SW423CT-ND" (id 6) (at 382.27 16.51 0)
-      (effects (font (size 1.27 1.27)) hide)
-    )
-    (property "Mouser PN" "N/A" (id 7) (at 382.27 13.97 0)
-      (effects (font (size 1.27 1.27)) hide)
-    )
-    (pin "1")
-    (pin "2")
-    (pin "3")
-    (pin "4")
-  )
   (symbol (lib_id "HPS:MountingHole") (at 35.56 271.78 0) (unit 1)
     (in_bom yes) (on_board yes)
@@
       (reference "#PWR010") (unit 1) (value "GND") (footprint "")
     )
-    (path "/c94a1b53-454d-4b3b-bee8-7a9b12abb405"
-      (reference "#PWR011") (unit 1) (value "VCC") (footprint "")
-    )
-    (path "/f0512e29-a102-44f3-884e-8f1468aa3327"
-      (reference "#PWR012") (unit 1) (value "GND") (footprint "")
-    )
     (path "/28b58255-5998-4ed5-b0e6-f11621736c10"
       (reference "#PWR013") (unit 1) (value "GND") (footprint "")
@@
       (reference "R4") (unit 1) (value "R_0805_47") (footprint "footprints:R_0805_2012Metric")
     )
-    (path "/94cec9dd-0011-4e74-8eac-76ffe61152fa"
-      (reference "R5") (unit 1) (value "R_0805_10K") (footprint "footprints:R_0805_2012Metric")
-    )
     (path "/07a93ead-2aa1-44f7-8a3f-0fa2ac6d6526"
       (reference "R6") (unit 1) (value "R_0805_10K") (footprint "footprints:R_0805_2012Metric")
@@
       (reference "SW1") (unit 1) (value "Omron_B3F_SPST") (footprint "footprints:SW_SPST_Omron_B3FS-100xP")
     )
-    (path "/fe3e14d0-07c3-41f7-84a8-2e1ac203c264"
-      (reference "SW3") (unit 1) (value "Omron_B3F_SPST") (footprint "footprints:SW_SPST_Omron_B3FS-100xP")
-    )
     (path "/9f3718d2-4c44-41a2-bdc9-fa0fdcd56d8e"
