File: Gitclock/Gitclock.kicad_pcb (KiCad board)
At the start: 2 copper layers, 140 x 90 mm, 4 parts

Commit message: gitclock6302022
Parts:
- added BZ1: Buzzer, footprints:Buzzer_TDK_PS1240P02BT_D12.2mm_H6.5mm, F.Cu at (129.5, 114.3)
- added C1: C_0805_0.1uf, footprints:C_0805_2012Metric, F.Cu at (115.8, 134.2)
- added C2: C_0805_0.1uf, footprints:C_0805_2012Metric, F.Cu at (203.3, 82.2)
- added C3: C_0805_0.1uf, footprints:C_0805_2012Metric, F.Cu at (124.6, 133.4)
- added C4: C_0805_22pf, footprints:C_0805_2012Metric, F.Cu at (141.1, 120.0)
- added C5: C_0805_22pf, footprints:C_0805_2012Metric, F.Cu at (141.8, 102.7)
- added C6: C_0805_1uf, footprints:C_0805_2012Metric, F.Cu at (152.2, 102.7)
- added C7: C_0805_0.1uf, footprints:C_0805_2012Metric, F.Cu at (146.2, 102.7)
- added D1: LED_0805, footprints:LED_0805_2012Metric, F.Cu at (94.8, 134.8)
- added DS1: LED_Display_1001, footprints:Adafruit-1001-0-0-MFG, F.Cu at (180.0, 89.2)
- added DS2: TC1602A-01T, footprints:TC1602A-01T, F.Cu at (96.2, 66.9)
- added J1: PJ-102AH, footprints:PJ-102AH, F.Cu at (115.2, 112.0)
- added J2: Conn_01x06, footprints:PinHeader_1x06_P2.54mm_Vertical, F.Cu at (203.4, 65.7)
- added J3: Conn_01x05, footprints:PinHeader_1x05_P2.54mm_Vertical, F.Cu at (122.6, 103.5)
- added R1: R_0805_2.2K, footprints:R_0805_2012Metric, F.Cu at (150.6, 105.6)
- added R11: R_0805_10K, footprints:R_0805_2012Metric, F.Cu at (124.6, 130.5)
- added R2: R_0805_10K, footprints:R_0805_2012Metric, F.Cu at (146.2, 105.6)
- added R3: R_0805_47, footprints:R_0805_2012Metric, F.Cu at (120.2, 134.2)
- added R4: R_0805_47, footprints:R_0805_2012Metric, F.Cu at (122.6, 117.5)
- added R5: R_0805_10K, footprints:R_0805_2012Metric, F.Cu at (141.8, 105.6)
- added R6: R_0805_10K, footprints:R_0805_2012Metric, F.Cu at (111.4, 134.2)
- added R8: R_0805_10K, footprints:R_0805_2012Metric, F.Cu at (133.8, 122.7)
- added R9: R_0805_10K, footprints:R_0805_2012Metric, F.Cu at (156.6, 102.7)
- added RV1: R_POT_10K, footprints:Potentiometer_Bourns_3386P_Vertical, F.Cu at (144.5, 115.5)
- added RV2: R_POT_10K, footprints:Potentiometer_Bourns_3386P_Vertical, F.Cu at (211.3, 71.4)
- added SW1: Omron_B3F_SPST, footprints:SW_SPST_Omron_B3FS-100xP, F.Cu at (126.0, 125.1)
- added SW2: Omron_B3F_SPST, footprints:SW_SPST_Omron_B3FS-100xP, F.Cu at (195.9, 104.4)
- added SW3: Omron_B3F_SPST, footprints:SW_SPST_Omron_B3FS-100xP, F.Cu at (114.8, 120.9)
- added SW4: Omron_B3F_SPST, footprints:SW_SPST_Omron_B3FS-100xP, F.Cu at (114.8, 128.8)
- added U1: ATmega328-PU, footprints:DIP-28_W7.62mm, F.Cu at (191.8, 65.4)
- added U3: MAX7219, footprints:DIP-24_W7.62mm, F.Cu at (89.1, 103.2)
- added U4: DS1307_DIP-8, footprints:DIP-8_W7.62mm, F.Cu at (99.9, 103.2)
- added U5: ULN2003A, footprints:DIP-16_W7.62mm, F.Cu at (99.9, 117.1)
- added Y1: Crystal_16MHz, footprints:Crystal_SMD_HC49-SD, F.Cu at (132.2, 104.3)
- added Y2: Crystal_32768Hz, footprints:Crystal_SMD_2Pin_3.2x1.5mm, F.Cu at (90.0, 135.0)
