File: Gitclock/Gitclock.kicad_pcb (KiCad board)
At the start: 2 copper layers, 140 x 90 mm, 39 parts, among them J1 PJ-102AH, J2 Conn_01x06, J3 Conn_01x05, SW1 Omron_B3F_SPST, SW2 Omron_B3F_SPST, SW3 Omron_B3F_SPST, SW4 Omron_B3F_SPST, U1 ATmega328-PU, U3 MAX7219, U4 DS1307_DIP-8, U5 ULN2003A, Y1 Crystal_16MHz, Y2 Crystal_32768Hz

Commit message: Gitclock
20220707
9:46AM
Parts:
- moved C6 133.3 mm to (283.6, 124.9)
- moved C3 133.3 mm to (256.0, 155.7)
- moved C4 133.3 mm to (272.5, 142.2)
- moved C5 133.3 mm to (273.2, 124.9)
- moved R1 133.3 mm to (282.0, 127.8)
- moved R11 133.3 mm to (256.0, 152.8)
- moved R4 133.3 mm to (254.0, 139.7)
- moved R5 133.3 mm to (273.2, 127.8)
- moved R8 133.3 mm to (265.2, 144.9)
- moved RV1 133.3 mm to (275.9, 137.8)
- moved C7 133.3 mm to (277.6, 124.9)
- moved R2 133.3 mm to (277.6, 127.8)
- moved R9 133.3 mm to (288.0, 124.9)
- moved J2 97.8 mm to (106.7, 80.0)
- moved U3 95.7 mm to (177.8, 67.3)
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
Commit message: Gitclock
20220707
3:55PM
Parts:
- removed R11: R_0805_10K, footprints:R_0805_2012Metric
- removed SW2, SW4: Omron_B3F_SPST, footprints:SW_SPST_Omron_B3FS-100xP
- added BT1: Battery_Cell, footprints:BatteryHolder_Keystone_106_1x20mm, F.Cu at (328.9, 124.5)
- added C8: C_0805_0.1uf, footprints:C_0805_2012Metric, F.Cu at (315.4, 136.4)
- added C9: C_0805_0.1uf, footprints:C_0805_2012Metric, F.Cu at (361.6, 134.7)
- added R10: R_0805_10K, footprints:R_0805_2012Metric, F.Cu at (357.2, 133.5)
- added R12: R_0805_10K, footprints:R_0805_2012Metric, F.Cu at (311.0, 136.4)
- added R13: R_0805_47, footprints:R_0805_2012Metric, F.Cu at (357.2, 136.4)
- added R7: R_0805_10K, footprints:R_0805_2012Metric, F.Cu at (337.1, 108.5)
- added SW5: RotaryEncoder_Switch, footprints:RotaryEncoder_TT_EN11-Switch_Vertical_H20mm_CircularMountingHoles, F.Cu at (357.0, 103.5)
- R8, R9: value R_0805_10K -> R_0805_4.7K
- moved U5 321.4 mm to (408.8, 62.0)
- moved U4 312.9 mm to (419.6, 62.0)
- moved J2 302.8 mm to (409.5, 84.2)
- moved R6 301.4 mm to (431.1, 64.4)
- moved J1 279.2 mm to (379.5, 108.6)
- moved BZ1 255.8 mm to (345.4, 104.7)
- moved DS1 249.6 mm to (396.9, 85.8), turned to 0 degrees
- moved J3 243.6 mm to (357.3, 116.6)
- moved RV2 233.4 mm to (376.4, 122.3)
- moved Y2 227.8 mm to (317.8, 131.6)
- moved SW1 218.9 mm to (412.8, 103.1)
- moved R3 209.0 mm to (357.2, 130.5)
- moved D1 208.5 mm to (328.4, 105.6)
- moved C3 202.7 mm to (435.5, 61.4)
- moved DS2 200.7 mm to (313.2, 63.5)
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Connections:
- BZ1 pad 2: FAN -> BUZZER
- C2 pad 1: VCC -> GND
- C7 pad 1: VCC -> GND
- D1 pad 2: SCK -> LED_SCK
- DS1 pad 7: unconnected-(DS1-Pad7) -> Net-(DS1-Pad7)
- DS1 pad 8: unconnected-(DS1-Pad8) -> Net-(DS1-Pad3)
- DS2 pad 1: unconnected-(DS2-Pad1) -> GND
- DS2 pad 11: unconnected-(DS2-Pad11) -> D4
- DS2 pad 12: unconnected-(DS2-Pad12) -> D5
- DS2 pad 13: unconnected-(DS2-Pad13) -> D6
- DS2 pad 14: unconnected-(DS2-Pad14) -> D7
- DS2 pad 15: unconnected-(DS2-Pad15) -> Net-(DS2-Pad15)
- DS2 pad 16: unconnected-(DS2-Pad16) -> GND
- DS2 pad 2: unconnected-(DS2-Pad2) -> GND
- DS2 pad 3: unconnected-(DS2-Pad3) -> Net-(DS2-Pad3)
- DS2 pad 4: unconnected-(DS2-Pad4) -> RS
- DS2 pad 5: unconnected-(DS2-Pad5) -> GND
- DS2 pad 6: unconnected-(DS2-Pad6) -> MOSI
- J3 pad 2: VCC -> Net-(J3-Pad2)
- R2 pad 1: VCC -> GND
- R5 pad 1: MENU -> GND
- R5 pad 2: GND -> FAN_B
- R6 pad 1: SNOOZE -> MENU SCROLL
- R8 pad 1: VCC -> GND
- R9 pad 1: VCC -> GND
- RV1 pad 1: VCC -> Net-(R12-Pad1)
- RV1 pad 2: unconnected-(RV1-Pad2) -> Net-(R12-Pad1)
- RV2 pad 1: MENU SCROLL -> GND
- RV2 pad 2: VCC -> Net-(DS2-Pad3)
- SW3 pad 1: VCC -> GND
- SW3 pad 3: MENU -> FAN_B
- U1 pad 11: unconnected-(U1-Pad11) -> D7
- U1 pad 12: BUZZER -> FAN
- U1 pad 13: MENU -> BUZZER
- U1 pad 14: SNOOZE -> LOAD
- U1 pad 15: FAN -> CLK
- U1 pad 16: SS -> DATA
- U1 pad 18: unconnected-(U1-Pad18) -> RS
- U1 pad 19: SCK -> LED_SCK
- U1 pad 20: VCC -> GND
- U1 pad 23: unconnected-(U1-Pad23) -> MENU SCROLL
- U1 pad 24: MENU SCROLL -> MENU OUTPUT2
- U1 pad 25: unconnected-(U1-Pad25) -> FAN_B
- U1 pad 26: unconnected-(U1-Pad26) -> MENU_B
- U1 pad 4: unconnected-(U1-Pad4) -> D4
- U1 pad 5: unconnected-(U1-Pad5) -> D5
- U1 pad 6: unconnected-(U1-Pad6) -> D6
- U1 pad 7: VCC -> GND
- U3 pad 1: MOSI -> DATA
- U3 pad 11: Net-(DS1-Pad14) -> Net-(DS1-Pad11)
- U3 pad 12: SS -> LOAD
- U3 pad 13: SCK -> CLK
- U3 pad 19: VCC -> GND
- U3 pad 2: unconnected-(U3-Pad2) -> Net-(DS1-Pad14)
- U3 pad 3: Net-(DS1-Pad6) -> Net-(DS1-Pad7)
- U3 pad 6: Net-(DS1-Pad11) -> Net-(DS1-Pad10)
- U3 pad 7: Net-(DS1-Pad10) -> Net-(DS1-Pad6)
- U4 pad 8: VCC -> GND
- U5 pad 1: Net-(SW4-Pad3) -> FAN
- U5 pad 9: VCC -> Net-(J3-Pad2)

Commit message: 20220713
5:40 PM clock
Parts:
- removed J3: Conn_01x05, footprints:PinHeader_1x05_P2.54mm_Vertical
- removed U5: ULN2003A, footprints:DIP-16_W7.62mm
- moved C4 317.7 mm to (104.1, 105.4), turned to 90 degrees
- moved U4 305.4 mm to (114.3, 68.6)
- moved R8 295.8 mm to (124.5, 74.9), turned to -90 degrees
- moved R6 295.6 mm to (135.9, 80.0)
- moved J1 281.4 mm to (99.1, 132.1)
- moved R5 280.1 mm to (130.8, 78.7), turned to 180 degrees
- moved RV2 249.2 mm to (128.3, 99.0), turned to 90 degrees
- moved R1 248.9 mm to (165.1, 80.0)
- moved R10 247.2 mm to (115.6, 81.3), turned to 180 degrees
- moved DS1 245.2 mm to (152.4, 67.3), turned to 90 degrees
- moved C6 245.0 mm to (88.9, 132.1), turned to 90 degrees
- moved C3 244.8 mm to (193.0, 95.2), turned to 180 degrees
- moved J2 242.1 mm to (167.6, 95.2), turned to 90 degrees
- moved BT1 240.0 mm to (95.2, 69.7), turned to -90 degrees
- moved BZ1 234.9 mm to (110.7, 95.2)
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Connections:
- net FAN_B renamed Select_B
- C2 pad 1: GND -> VCC
- C7 pad 1: GND -> VCC
- C8 pad 1: GND -> VCC
- C9 pad 1: GND -> VCC
- DS2 pad 2: GND -> VCC
- R12 pad 2: GND -> VCC
- R13 pad 2: GND -> VCC
- R2 pad 1: GND -> VCC
- R8 pad 1: GND -> VCC
- R9 pad 1: GND -> VCC
- RV2 pad 3: GND -> VCC
- SW3 pad 1: GND -> VCC
- SW5 pad S1: GND -> VCC
- U1 pad 12: FAN -> unconnected-(U1-Pad12)
- U1 pad 20: GND -> VCC
- U1 pad 7: GND -> VCC
- U3 pad 19: GND -> VCC
- U4 pad 8: GND -> VCC

Commit message: 0719clock
Parts:
- BT1: moved to B.Cu
- moved R2 130.2 mm to (91.4, 66.0)
- moved SW5 108.0 mm to (89.3, 114.3)
- moved R7 106.3 mm to (86.7, 114.3)
- moved R10 101.2 mm to (214.6, 102.0), turned to 90 degrees
- moved BZ1 86.2 mm to (196.7, 90.2), turned to 180 degrees
- moved C2 80.5 mm to (91.4, 74.9)
- moved R5 78.5 mm to (193.0, 126.6), turned to -90 degrees
- moved C8 69.2 mm to (130.8, 92.7), turned to -90 degrees
- moved R6 64.5 mm to (83.8, 118.1), turned to 90 degrees
- moved Y1 54.1 mm to (90.2, 86.4), turned to 90 degrees
- moved R1 52.5 mm to (113.0, 86.4), turned to 90 degrees
- moved BT1 48.9 mm to (108.1, 116.8), turned to 180 degrees
- moved J2 47.6 mm to (200.7, 61.0), turned to 0 degrees
- moved C5 47.1 mm to (90.2, 97.8), turned to -90 degrees
- moved C1 46.0 mm to (108.0, 83.8), turned to 0 degrees
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Routing:
- net BUZZER: track 0.00 -> 115.9 mm, vias 0 -> 1
- net GND: track 0.00 -> 87.9 mm, vias 0 -> 7
- net CLK: track 0.00 -> 72.0 mm
- net Net-(DS1-Pad11): track 0.00 -> 43.7 mm, vias 0 -> 2
- net Net-(DS1-Pad13): track 0.00 -> 39.4 mm, vias 0 -> 2
- net Net-(DS1-Pad12): track 0.00 -> 34.3 mm, vias 0 -> 2
- net RS: track 0.00 -> 33.0 mm, vias 0 -> 1
- net Net-(DS1-Pad14): track 0.00 -> 32.1 mm
- net Net-(DS1-Pad7): track 0.00 -> 30.3 mm, vias 0 -> 1
- net Net-(RV1-Pad3): track 0.00 -> 28.0 mm
- net Net-(DS1-Pad9): track 0.00 -> 23.4 mm
- net RESET: track 0.00 -> 19.3 mm
- net Net-(DS1-Pad2): track 0.00 -> 19.0 mm, vias 0 -> 1
- net SDA: track 0.00 -> 18.7 mm
- net SCL: track 0.00 -> 18.7 mm
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- added copper zone on B.Cu, net GND
- added copper zone on B.Cu, net VCC
- added copper zone on F.Cu, net VCC

Commit message: Routing display
Parts:
- J2: moved to B.Cu
- moved R10 108.1 mm to (106.7, 108.0)
- moved J2 108.0 mm to (92.7, 59.7), turned to -90 degrees
- moved BT1 97.0 mm to (203.2, 97.8), turned to -90 degrees
- moved R3 94.1 mm to (99.1, 63.5)
- moved C3 88.1 mm to (102.9, 63.5)
- moved R6 2.54 mm to (86.4, 118.1)
- moved R8 1.27 mm to (106.7, 68.6)
- moved R9 1.27 mm to (106.7, 63.5)
- moved U4 1.27 mm to (113.0, 59.7)
- moved Y2 1.27 mm to (109.2, 61.0)
- moved R7 0.37 mm to (86.4, 114.3)
Routing:
- net +BATT: track 0.00 -> 136.2 mm
- net MENU OUTPUT2: track 0.00 -> 50.2 mm
- net GND: track 87.9 -> 50.7 mm, vias 7 -> 5
- net Net-(C3-Pad2): track 9.84 -> 0.00 mm
- net RESET: track 19.3 -> 11.0 mm
- net Net-(J2-Pad5): track 7.82 -> 0.00 mm
- net MENU_B: track 0.00 -> 6.75 mm
- net BUZZER: track 115.9 -> 109.3 mm
- net MENU SCROLL: track 0.00 -> 3.07 mm

Commit message: Final Routing Pass
Parts:
- removed R5: R_0805_10K, footprints:R_0805_2012Metric
- removed SW3: Omron_B3F_SPST, footprints:SW_SPST_Omron_B3FS-100xP
- added U2: L7805, footprints:TO-252-2, F.Cu at (192.2, 73.4)
- J1: moved to B.Cu
- moved J1 123.3 mm to (206.7, 71.6)
- moved C7 111.5 mm to (194.3, 67.3), turned to 180 degrees
- moved C6 100.2 mm to (193.0, 80.0), turned to 180 degrees
- moved C9 21.3 mm to (148.6, 86.4), turned to 0 degrees
- moved C3 18.9 mm to (85.1, 69.8), turned to 180 degrees
- moved C8 15.3 mm to (144.8, 86.4), turned to 180 degrees
- moved R2 6.48 mm to (85.1, 67.3)
- moved R4 3.81 mm to (91.4, 64.8), turned to 0 degrees
Routing:
- net D6: track 0.00 -> 87.7 mm, vias 0 -> 2
- net D5: track 0.00 -> 85.1 mm, vias 0 -> 2
- net D4: track 0.00 -> 84.1 mm, vias 0 -> 2
- net D7: track 0.00 -> 78.4 mm, vias 0 -> 2
- net LOAD: track 0.00 -> 75.2 mm, vias 0 -> 1
- net MENU_B: track 6.75 -> 54.9 mm, vias 0 -> 2
- net MENU SCROLL: track 3.07 -> 50.9 mm
- net MOSI: track 0.00 -> 38.1 mm, vias 0 -> 1
- net DATA: track 0.00 -> 31.7 mm
- net Net-(C3-Pad2): track 0.00 -> 30.3 mm, vias 0 -> 1
- net Net-(DS2-Pad3): track 0.00 -> 13.2 mm
- net Net-(J2-Pad4): track 0.00 -> 10.1 mm
- net RESET: track 11.0 -> 20.4 mm
- net +BATT: track 136.2 -> 145.3 mm
- net TXD: track 0.00 -> 8.85 mm
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- removed copper zone on B.Cu, net VCC
