File: Gitclock/_autosave-Gitclock.kicad_pcb (KiCad board)
At the start: 2 copper layers, 140 x 90 mm, 42 parts, among them J1 PJ-102AH, J2 Conn_01x06, SW1 Omron_B3F_SPST, SW3 Omron_B3F_SPST, SW5 RotaryEncoder_Switch, U1 ATmega328-PU, U3 MAX7219, U4 DS1307_DIP-8, Y1 Crystal_16MHz, Y2 Crystal_32768Hz

Commit message: Routing display
Parts:
- added U2: L7805, footprints:TO-252-2, F.Cu at (192.2, 73.4)
- J1: moved to B.Cu
- moved J1 123.3 mm to (206.7, 71.6)
- moved C7 111.5 mm to (194.3, 67.3), turned to 180 degrees
- moved C6 100.2 mm to (193.0, 80.0), turned to 180 degrees
Routing:
- net GND: track 50.7 -> 38.0 mm
- net +BATT: track 136.2 -> 145.3 mm
- net Net-(C6-Pad1): track 7.36 -> 14.7 mm
